Commit message: feat: Added Gazebo diff drive and joint state publisher plugins

File: xacro/castor_wheels.xacro (robot description, xacro)
@@ -9,5 +9,25 @@
                 </geometry>
             </visual>
+            <inertial>
+                <mass value="0.7"/>
+                <origin xyz=" 0 0 0" rpy="0 0 0" />
+                <inertia ixx="0.0020" ixy="0" ixz="0"
+                        iyx="0" iyy="0.0020" iyz="0"
+                        izx="0" izy="0" izz="0.0025" />
+            </inertial>
+            <collision>
+                <origin xyz="0 0 0" rpy="0 0 0"/>
+                <geometry>
+                    <cylinder length="0.01" radius="0.05"/>
+                </geometry>
+            </collision>
         </link>
+        <gazebo reference="${prefix}_castor_wheel_yaw_link">
+            <material>Gazebo/Black</material>
+            <mu1>100</mu1>
+            <mu2>100</mu2>
+            <kp>100000000000000000</kp>
+            <kd>100000000000000000</kd>
+        </gazebo>
         <joint name="${prefix}_castor_wheel_yaw_joint" type="continuous">
             <parent link="${parent}"/>
@@ -15,4 +35,6 @@
             <origin xyz="${castor_base_xoff} ${y_reflect * castor_base_yoff} 0" rpy="0 0 0"/>
             <axis xyz="0 0 1"/>
+            <limit effort="100" velocity="100"/>
+            <dynamics damping="1.0" friction="10.0"/>
         </joint>
         <link name="${prefix}_castor_wheel_base_link">
@@ -23,5 +45,25 @@
                 </geometry>
             </visual>
+            <inertial>
+                <mass value="0.7"/>
+                <origin xyz="0 0 0" rpy="0 ${1.57/2} 0"/>
+                <inertia ixx="0.0015" ixy="0" ixz="0"
+                        iyx="0" iyy="0.0012" iyz="0"
+                        izx="0" izy="0" izz="0.0017" />
+            </inertial>
+            <collision>
+                <origin xyz="0 0 0" rpy="0 ${1.57/2} 0"/>
+                <geometry>
+                    <box size="0.03 0.03 ${-castor_center_xoff/0.7}"/>
+                </geometry>
+            </collision>
         </link>
+        <gazebo reference="${prefix}_castor_wheel_base_link">
+            <material>Gazebo/Red</material>
+            <mu1>100</mu1>
+            <mu2>100</mu2>
+            <kp>100000000000000000</kp>
+            <kd>100000000000000000</kd>
+        </gazebo>
         <joint name="${prefix}_castor_wheel_base_joint" type="fixed">
             <parent link="${prefix}_castor_wheel_yaw_link"/>
@@ -38,5 +80,25 @@
                 </geometry>
             </visual>
+            <inertial>
+                <mass value="1.0"/>
+                <origin xyz=" 0 0 0" rpy="0 0 0" />
+                <inertia ixx="0.0020" ixy="0" ixz="0"
+                        iyx="0" iyy="0.0025" iyz="0"
+                        izx="0" izy="0" izz="0.0020" />
+            </inertial>
+            <collision>
+                <origin xyz="0 0 0" rpy="1.57 0 0"/>
+                <geometry>
+                    <cylinder length="${castor_wheel_width}" radius="${castor_wheel_radius}"/>
+                </geometry>
+            </collision>
         </link>
+        <gazebo reference="${prefix}_castor_wheel_pitch_link">
+            <material>Gazebo/Red</material>
+            <mu1>50</mu1>
+            <mu2>50</mu2>
+            <kp>10000000</kp>
+            <kd>10000000</kd>
+        </gazebo>
         <joint name="${prefix}_castor_wheel_pitch_joint" type="continuous">
             <parent link="${prefix}_castor_wheel_base_link"/>
@@ -46,4 +108,6 @@
                          ${castor_center_zoff/2}" rpy="0 0 0"/>
             <axis xyz="0 1 0"/>
+            <limit effort="1000" velocity="1000"/>
+            <dynamics damping="1.0" friction="10.0"/>
         </joint>
     </xacro:macro>

File: xacro/properties.xacro (robot description, xacro)
@@ -2,5 +2,5 @@
 <robot xmlns:xacro="http://ros.org/wiki/xacro">
     <!-- General constants -->
-    <xacro:property name="vikings_bot_mass" value="50.0"/>
+    <xacro:property name="vikings_bot_mass" value="60.0"/>
     <xacro:property name="vikings_bot_x" value="1.0"/>
     <xacro:property name="vikings_bot_y" value="0.68"/>
@@ -15,5 +15,5 @@
     <xacro:property name="castor_base_xoff" value="0.31"/>
     <xacro:property name="castor_base_yoff" value="0.2725"/>
-    <xacro:property name="castor_base_zoff" value="0.005"/>
+    <xacro:property name="castor_base_zoff" value="0.015"/>
     <xacro:property name="castor_center_xoff" value="-0.052"/>
     <xacro:property name="castor_center_yoff" value="0.0"/>

File: xacro/test.urdf (robot description, URDF)
Before this commit: robot vikings_bot, 12 links, 11 joints
Links:
- added link camera_link, mass 0.2; collision box size=0.08 0.1 0.03; visual mesh filename=package://vikings_bot_description/meshes/sensors/realsense.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 scale=1 1 1
- added link dummy_link, mass 0.05
- link base_link: mass None -> 0.05
- link chassis_link: mass None -> 60; geometry collision box size=1.0 0.68 0.24; visual box size=1.0 0.68 0.24
- link left_castor_wheel_base_link: mass None -> 0.7; geometry collision box size=0.03 0.03 0.07428571428571429; visual box size=0.03 0.03 0.07428571428571429
- link left_castor_wheel_pitch_link: mass None -> 1.0; geometry collision cylinder length=0.05 radius=0.0612; visual cylinder length=0.05 radius=0.0612
- link left_castor_wheel_yaw_link: mass None -> 0.7; geometry collision cylinder length=0.01 radius=0.05; visual cylinder length=0.01 radius=0.05
- link left_drive_wheel_link: mass None -> 5; geometry collision cylinder length=0.05 radius=0.125; visual cylinder length=0.05 radius=0.125
- link lidar_link: mass None -> 0.2; geometry collision box size=0.08 0.08 0.08; visual mesh filename=package://vikings_bot_description/meshes/sensors/rplidar.dae scale=1 1 1
- link right_castor_wheel_base_link: mass None -> 0.7; geometry collision box size=0.03 0.03 0.07428571428571429; visual box size=0.03 0.03 0.07428571428571429
- link right_castor_wheel_pitch_link: mass None -> 1.0; geometry collision cylinder length=0.05 radius=0.0612; visual cylinder length=0.05 radius=0.0612
- link right_castor_wheel_yaw_link: mass None -> 0.7; geometry collision cylinder length=0.01 radius=0.05; visual cylinder length=0.01 radius=0.05
- link right_drive_wheel_link: mass None -> 5; geometry collision cylinder length=0.05 radius=0.125; visual cylinder length=0.05 radius=0.125
Joints:
- added joint camera_link_joint: type fixed, parent chassis_link, child camera_link, origin xyz=0.5 0.0 0.06 rpy=0 0 0
- added joint chassis_joint: type fixed, parent dummy_link, child chassis_link, origin xyz=0 0 -0.155 rpy=0 0 0
- joint left_castor_wheel_pitch_joint: limit (none) -> effort=1000 velocity=1000
- joint left_castor_wheel_yaw_joint: limit (none) -> effort=100 velocity=100
- joint left_drive_wheel_joint: limit (none) -> effort=1000 velocity=1000
- joint lidar_link_joint: origin xyz=1 0 0 rpy=0 0 0 -> xyz=0.53 0.0 -0.06 rpy=0 0 0
- joint right_castor_wheel_pitch_joint: limit (none) -> effort=1000 velocity=1000
- joint right_castor_wheel_yaw_joint: limit (none) -> effort=100 velocity=100
- joint right_drive_wheel_joint: limit (none) -> effort=1000 velocity=1000

File: xacro/vikings_bot.xacro (robot description, xacro)
@@ -3,6 +3,8 @@
     <!-- Argumnets -->
     <xacro:arg name="vikings_bot_name" default="vikings_bot"/>
+    <xacro:arg name="use_gazebo" default="yes"/>
     <!-- Robot properties -->
     <xacro:property name="robot_name" value="$(arg vikings_bot_name)"/>
+    <xacro:property name="use_gazebo" value="$(arg use_gazebo)"/>
     <!-- Include robot properties -->
     <xacro:include filename="$(find vikings_bot_description)/xacro/properties.xacro"/>
@@ -12,6 +14,18 @@
     <xacro:include filename="$(find vikings_bot_description)/xacro/wheels.xacro"/>
     <xacro:include filename="$(find vikings_bot_description)/xacro/castor_wheels.xacro"/>
+    <!-- Inlude gazebo stuff -->
+    <!-- <xacro:include filename="$(find vikings_bot_description)/xacro/gazebo_plugins.xacro"/> -->
     <!-- Include Gazebo related files -->
     <!-- ROBOT -->
+    <!-- Dummy link -->
+    <link name="${robot_name}dummy_link">
+        <inertial>
+            <mass value="0.05"/>
+            <origin xyz=" 0 0 0" rpy="0 0 0" />
+            <inertia ixx="0" ixy="0" ixz="0"
+                     iyx="0" iyy="0" iyz="0"
+                     izx="0" izy="0" izz="0" />
+        </inertial>
+    </link>
     <!-- Chassis link-->
     <link name="chassis_link">
@@ -22,5 +36,35 @@
             <material name="blue"/>
         </visual>
-    </link>
+        <inertial>
+            <mass value="${vikings_bot_mass}"/>
+            <origin xyz=" 0 0 0" rpy="0 0 0" />
+            <inertia ixx="2.6245" ixy="0" ixz="0"
+                     iyx="0" iyy="5.3125" iyz="0"
+                     izx="0" izy="0" izz="7.3120" />
+        </inertial>
+        <collision>
+            <geometry>
+                <box size="${vikings_bot_x} ${vikings_bot_y} ${vikings_bot_z}"/>
+            </geometry>
+        </collision>
+    </link>
+    <gazebo reference="chassis_link">
+        <material>Gazebo/Blue</material>
+        <!-- friction -->
+        <mu1>100</mu1>
+        <mu2>100</mu2>
+        <!-- stiffness -->
+        <kp>100000000000000000</kp>
+        <kd>100000000000000000</kd>
+    </gazebo>
+    <!-- Chassis joint-->
+    <joint name="chassis_joint" type="fixed">
+        <parent link="dummy_link"/>
+        <child link="chassis_link"/>
+        <origin xyz="0 0 ${-(wheel_radius-wheel_zoff)}" rpy="0 0 0"/>
+    </joint>
+    <gazebo reference="chassis_joint">
+        <preserveFixedJoint>true</preserveFixedJoint>
+    </gazebo>
     <!-- Footprint link-->
     <link name="base_footprint_link"/>
@@ -31,6 +75,17 @@
         <origin xyz="0 0 ${-(wheel_radius-wheel_zoff)}" rpy="0 0 0"/>
     </joint>
+    <gazebo reference="base_footprint_joint">
+        <preserveFixedJoint>true</preserveFixedJoint>
+    </gazebo>
     <!-- Base link-->
-    <link name="base_link"/>
+    <link name="base_link">
+        <inertial>
+            <mass value="0.1"/>
+            <!-- <origin xyz=" 0 0 0" rpy="0 0 0" />
+            <inertia ixx="0" ixy="0" ixz="0"
+                     iyx="0" iyy="0" iyz="0"
+                     izx="0" izy="0" izz="0" />    -->
+        </inertial>
+    </link>
     <!-- Base link joint -->
     <joint name="base_link_joint" type="fixed">
@@ -39,4 +94,7 @@
         <origin xyz="${wheel_xoff} 0 ${wheel_zoff}" rpy="0 0 0"/>
     </joint>
+    <gazebo reference="base_link_joint">
+        <preserveFixedJoint>true</preserveFixedJoint>
+    </gazebo>
     <!-- Drive wheels -->
     <xacro:drive_wheel prefix="left" parent="base_link" y_reflect="1.0"/>
@@ -54,5 +112,27 @@
             </geometry>
         </visual>
-    </link>
+        <inertial>
+            <mass value="0.2"/>
+            <origin xyz=" 0 0 0" rpy="0 0 0" />
+            <inertia ixx="1e-7" ixy="0" ixz="0"
+                     iyx="0" iyy="1e-7" iyz="0"
+                     izx="0" izy="0" izz="1e-7" />
+        </inertial>
+        <collision>
+            <origin xyz="0 0 0.03" rpy="0 0 0"/>
+            <geometry>
+                <box size="0.08 0.08 0.08"/>
+            </geometry>
+        </collision>
+    </link>
+    <gazebo reference="lidar_link">
+        <material>Gazebo/Grey</material>
+        <!-- friction -->
+        <mu1>100</mu1>
+        <mu2>100</mu2>
+        <!-- stiffness -->
+        <kp>100000000000000000</kp>
+        <kd>100000000000000000</kd>
+    </gazebo>
     <joint name="lidar_link_joint" type="fixed">
         <parent link="chassis_link"/>
@@ -69,5 +149,26 @@
             </geometry>
         </visual>
-    </link>
+        <inertial>
+            <mass value="0.2"/>
+            <origin xyz=" 0 0 0" rpy="0 0 0" />
+            <inertia ixx="1e-7" ixy="0" ixz="0"
+                     iyx="0" iyy="1e-7" iyz="0"
+                     izx="0" izy="0" izz="1e-7" />
+        </inertial>
+        <collision>
+            <geometry>
+                <box size="0.08 0.1 0.03"/>
+            </geometry>
+        </collision>
+    </link>
+    <gazebo reference="camera_link">
+        <material>Gazebo/Grey</material>
+        <!-- friction -->
+        <mu1>100</mu1>
+        <mu2>100</mu2>
+        <!-- stiffness -->
+        <kp>100000000000000000</kp>
+        <kd>100000000000000000</kd>
+    </gazebo>
     <joint name="camera_link_joint" type="fixed">
         <parent link="chassis_link"/>
@@ -75,3 +176,46 @@
         <origin xyz="${camera_xoff} ${camera_yoff} ${camera_zoff}" rpy="0 0 0"/>
     </joint>
+    <!-- PLUGINS -->
+    <gazebo>
+        <plugin name="${robot_name}_joint_state" filename="libgazebo_ros_joint_state_publisher.so">
+            <ros>
+                <namespace>/${robot_name}</namespace>
+                <!-- <remapping>~/out:=joint_states</remapping> -->
+            </ros>
+            <update_rate>30</update_rate>
+            <joint_name>left_drive_wheel_joint</joint_name>
+            <joint_name>right_drive_wheel_joint</joint_name>
+            <joint_name>left_castor_wheel_yaw_joint</joint_name>
+            <joint_name>right_castor_wheel_yaw_joint</joint_name>
+            <joint_name>left_castor_wheel_pitch_joint</joint_name>
+            <joint_name>right_castor_wheel_pitch_joint</joint_name>
+        </plugin>
+    </gazebo>
+    <!-- Differential drive -->
+    <gazebo>
+        <plugin filename="libgazebo_ros_diff_drive.so" name="${robot_name}_differential_drive_controller">
+        <ros>
+            <namespace>/${robot_name}</namespace>
+            <!--
+    <argument> -ros-args -remap /cmd_vel:=/${robot_name}/cmd_vel /odom:=/${robot_name}/odom</argument>
+-->
+        </ros>
+        <!-- wheels -->
+        <!-- wheels RMF COMPAT -->
+        <left_joint>left_drive_wheel_joint</left_joint>
+        <right_joint>right_drive_wheel_joint</right_joint>
+        <!-- kinematics -->
+        <wheel_separation>${wheel_yoff * 2}</wheel_separation>
+        <wheel_diameter>${wheel_radius * 2}</wheel_diameter>
+        <!-- limits -->
+        <max_wheel_torque>10000</max_wheel_torque>
+        <max_wheel_acceleration>1000</max_wheel_acceleration>
+        <!-- output -->
+        <publish_odom>true</publish_odom>
+        <publish_odom_tf>true</publish_odom_tf>
+        <!-- <publish_wheel_tf>false</publish_wheel_tf> -->
+        <odometry_frame>${robot_name}/odom</odometry_frame>
+        <robot_base_frame>${robot_name}/dummy_link</robot_base_frame>
+        </plugin>
+    </gazebo>
 </robot>

File: xacro/wheels.xacro (robot description, xacro)
@@ -9,5 +9,27 @@
                 </geometry>
             </visual>
+            <inertial>
+                <mass value="5"/>
+                <origin xyz=" 0 0 0" rpy="0 0 0" />
+                <inertia ixx="0.0206" ixy="0" ixz="0"
+                        iyx="0" iyy="0.0390" iyz="0"
+                        izx="0" izy="0" izz="0.0206" />
+            </inertial>
+            <collision>
+                <origin xyz="0 0 0" rpy="1.57 0 0"/>
+                <geometry>
+                    <cylinder length="${wheel_width}" radius="${wheel_radius}"/>
+                </geometry>
+            </collision>
         </link>
+        <gazebo reference="${prefix}_drive_wheel_link">
+            <material>Gazebo/Red</material>
+            <!-- friction -->
+            <mu1>10</mu1>
+            <mu2>10</mu2>
+            <!-- stiffness -->
+            <kp>1000000</kp>
+            <kd>1000000</kd>
+        </gazebo>
         <joint name="${prefix}_drive_wheel_joint" type="continuous">
             <parent link="${parent}"/>
@@ -16,4 +38,6 @@
             <origin xyz="0 ${y_reflect * wheel_yoff} 0" rpy="0 0 0"/>
             <axis xyz="0 1 0"/>
+            <limit effort="1000" velocity="1000"/>
+            <dynamics damping="1.0" friction="10.0"/>
         </joint>
     </xacro:macro>

Commit message: fix: removed continous joint property from catsor wheels

File: xacro/castor_wheels.xacro (robot description, xacro)
@@ -30,5 +30,5 @@
             <kd>100000000000000000</kd>
         </gazebo>
-        <joint name="${prefix}_castor_wheel_yaw_joint" type="continuous">
+        <joint name="${prefix}_castor_wheel_yaw_joint" type="fixed">
             <parent link="${parent}"/>
             <child link="${prefix}_castor_wheel_yaw_link"/>
@@ -96,10 +96,10 @@
         <gazebo reference="${prefix}_castor_wheel_pitch_link">
             <material>Gazebo/Red</material>
-            <mu1>50</mu1>
-            <mu2>50</mu2>
-            <kp>10000000</kp>
-            <kd>10000000</kd>
+            <mu1>0.01</mu1>
+            <mu2>0.01</mu2>
+            <kp>100000000000</kp>
+            <kd>100000000000</kd>
         </gazebo>
-        <joint name="${prefix}_castor_wheel_pitch_joint" type="continuous">
+        <joint name="${prefix}_castor_wheel_pitch_joint" type="fixed">
             <parent link="${prefix}_castor_wheel_base_link"/>
             <child link="${prefix}_castor_wheel_pitch_link"/>

File: xacro/wheels.xacro (robot description, xacro)
@@ -29,6 +29,6 @@
             <mu2>10</mu2>
             <!-- stiffness -->
-            <kp>1000000</kp>
-            <kd>1000000</kd>
+            <kp>10000000</kp>
+            <kd>10000000</kd>
         </gazebo>
         <joint name="${prefix}_drive_wheel_joint" type="continuous">

Commit message: feat: chnaged collision geometry for wheels

File: xacro/castor_wheels.xacro (robot description, xacro)
@@ -90,5 +90,6 @@
                 <origin xyz="0 0 0" rpy="1.57 0 0"/>
                 <geometry>
-                    <cylinder length="${castor_wheel_width}" radius="${castor_wheel_radius}"/>
+                    <!-- <cylinder length="${castor_wheel_width}" radius="${castor_wheel_radius}"/> -->
+                    <sphere radius="${castor_wheel_radius}"/>
                 </geometry>
             </collision>
@@ -96,8 +97,8 @@
         <gazebo reference="${prefix}_castor_wheel_pitch_link">
             <material>Gazebo/Red</material>
-            <mu1>0.01</mu1>
-            <mu2>0.01</mu2>
-            <kp>100000000000</kp>
-            <kd>100000000000</kd>
+            <mu1>0.001</mu1>
+            <mu2>0.001</mu2>
+            <!-- <kp>100000000000</kp>
+            <kd>100000000000</kd> -->
         </gazebo>
         <joint name="${prefix}_castor_wheel_pitch_joint" type="fixed">

File: xacro/wheels.xacro (robot description, xacro)
@@ -19,5 +19,6 @@
                 <origin xyz="0 0 0" rpy="1.57 0 0"/>
                 <geometry>
-                    <cylinder length="${wheel_width}" radius="${wheel_radius}"/>
+                    <!-- <cylinder length="${wheel_width}" radius="${wheel_radius}"/> -->
+                    <sphere radius="${wheel_radius}"/>
                 </geometry>
             </collision>
@@ -26,9 +27,9 @@
             <material>Gazebo/Red</material>
             <!-- friction -->
-            <mu1>10</mu1>
-            <mu2>10</mu2>
+            <!-- <mu1>100</mu1>
+            <mu2>100</mu2> -->
             <!-- stiffness -->
-            <kp>10000000</kp>
-            <kd>10000000</kd>
+            <!-- <kp>10000000</kp>
+            <kd>10000000</kd> -->
         </gazebo>
         <joint name="${prefix}_drive_wheel_joint" type="continuous">
@@ -39,5 +40,5 @@
             <axis xyz="0 1 0"/>
             <limit effort="1000" velocity="1000"/>
-            <dynamics damping="1.0" friction="10.0"/>
+            <!-- <dynamics damping="1.0" friction="10.0"/> -->
         </joint>
     </xacro:macro>
