Commit message: fix: repaired robot xacro file

File: xacro/gazebo_control.xacro (robot description, xacro)
@@ -41,5 +41,5 @@
         <!-- <publish_wheel_tf>false</publish_wheel_tf> -->
         <odometry_frame>${robot_name}/odom</odometry_frame>
-        <robot_base_frame>${robot_name}/dummy_link</robot_base_frame>
+        <robot_base_frame>${robot_name}/base_link</robot_base_frame>
         </plugin>
     </gazebo>

File: xacro/vikings_bot.xacro (robot description, xacro)
@@ -16,6 +16,6 @@
     <!-- Include Gazebo related files -->
     <!-- ROBOT -->
-    <!-- Dummy link -->
-    <link name="dummy_link">
+    <!-- Base link -->
+    <link name="base_link">
         <inertial>
             <mass value="0.05"/>
@@ -58,7 +58,8 @@
     <!-- Chassis joint-->
     <joint name="chassis_joint" type="fixed">
-        <parent link="dummy_link"/>
+        <parent link="base_link"/>
         <child link="chassis_link"/>
-        <origin xyz="0 0 0" rpy="0 0 0"/>
+        <!-- <origin xyz="0 0 0" rpy="0 0 0"/> -->
+        <origin xyz="${-(wheel_xoff)} 0 ${-(wheel_zoff)}" rpy="0 0 0"/>
     </joint>
     <gazebo reference="chassis_joint">
@@ -69,28 +70,9 @@
     <!-- Footprint joint -->
     <joint name="base_footprint_joint" type="fixed">
-        <parent link="chassis_link"/>
+        <parent link="base_link"/>
         <child link="base_footprint_link"/>
         <origin xyz="0 0 ${-(wheel_radius-wheel_zoff)}" rpy="0 0 0"/>
     </joint>
     <gazebo reference="base_footprint_joint">
-        <preserveFixedJoint>true</preserveFixedJoint>
-    </gazebo>
-    <!-- Base link-->
-    <link name="base_link">
-        <inertial>
-            <mass value="0.1"/>
-            <origin xyz=" 0 0 0" rpy="0 0 0" />
-            <inertia ixx="0" ixy="0" ixz="0"
-                     iyx="0" iyy="0" iyz="0"
-                     izx="0" izy="0" izz="0" />
-        </inertial>
-    </link>
-    <!-- Base link joint -->
-    <joint name="base_link_joint" type="fixed">
-        <parent link="chassis_link"/>
-        <child link="base_link"/>
-        <origin xyz="${wheel_xoff} 0 ${wheel_zoff}" rpy="0 0 0"/>
-    </joint>
-    <gazebo reference="base_link_joint">
         <preserveFixedJoint>true</preserveFixedJoint>
     </gazebo>
