Commit message: feat: added launch arguments to spawn mutiple robots with namespaces

File: xacro/vikings_bot.xacro (robot description, xacro)
@@ -19,5 +19,5 @@
     <!-- ROBOT -->
     <!-- Dummy link -->
-    <link name="${robot_name}dummy_link">
+    <link name="dummy_link">
         <inertial>
             <mass value="0.05"/>
@@ -62,5 +62,5 @@
         <parent link="dummy_link"/>
         <child link="chassis_link"/>
-        <origin xyz="0 0 ${-(wheel_radius-wheel_zoff)}" rpy="0 0 0"/>
+        <origin xyz="0 0 0" rpy="0 0 0"/>
     </joint>
     <gazebo reference="chassis_joint">
@@ -82,8 +82,8 @@
         <inertial>
             <mass value="0.1"/>
-            <!-- <origin xyz=" 0 0 0" rpy="0 0 0" />
+            <origin xyz=" 0 0 0" rpy="0 0 0" />
             <inertia ixx="0" ixy="0" ixz="0"
                      iyx="0" iyy="0" iyz="0"
-                     izx="0" izy="0" izz="0" />    -->
+                     izx="0" izy="0" izz="0" />
         </inertial>
     </link>

Commit message: add realsense plugin and model

File: xacro/vikings_bot.xacro (robot description, xacro)
@@ -14,4 +14,5 @@
     <xacro:include filename="$(find vikings_bot_description)/xacro/wheels.xacro"/>
     <xacro:include filename="$(find vikings_bot_description)/xacro/castor_wheels.xacro"/>
+    <xacro:include filename="$(find realsense2_description)/urdf/_d435i.urdf.xacro"/>
     <!-- Inlude gazebo stuff -->
     <!-- <xacro:include filename="$(find vikings_bot_description)/xacro/gazebo_plugins.xacro"/> -->
@@ -127,5 +128,5 @@
     </link>
     <gazebo reference="lidar_link">
-        <material>Gazebo/Grey</material>
+        <material>Gazebo/DarkGrey</material>
         <!-- friction -->
         <mu1>100</mu1>
@@ -141,25 +142,7 @@
     </joint>
     <!-- Camera -->
-    <link name="camera_link">
-        <visual>
-            <origin xyz="0 0 0" rpy="0 0 ${1.57*2}"/>
-            <geometry>
-                <mesh filename="package://vikings_bot_description/meshes/sensors/realsense.dae"
-                      scale="1 1 1"/>
-            </geometry>
-        </visual>
-        <inertial>
-            <mass value="0.2"/>
-            <origin xyz=" 0 0 0" rpy="0 0 0" />
-            <inertia ixx="1e-7" ixy="0" ixz="0"
-                     iyx="0" iyy="1e-7" iyz="0"
-                     izx="0" izy="0" izz="1e-7" />
-        </inertial>
-        <collision>
-            <geometry>
-                <box size="0.08 0.1 0.03"/>
-            </geometry>
-        </collision>
-    </link>
+    <xacro:sensor_d435i parent="chassis_link" use_nominal_extrinsics="true">
+        <origin xyz="${camera_xoff} ${camera_yoff} ${camera_zoff}" rpy="0 0 0"/>
+    </xacro:sensor_d435i>
     <gazebo reference="camera_link">
         <material>Gazebo/Grey</material>
@@ -171,9 +154,4 @@
         <kd>100000000000000000</kd>
     </gazebo>
-    <joint name="camera_link_joint" type="fixed">
-        <parent link="chassis_link"/>
-        <child link="camera_link"/>
-        <origin xyz="${camera_xoff} ${camera_yoff} ${camera_zoff}" rpy="0 0 0"/>
-    </joint>
     <!-- PLUGINS -->
     <gazebo>
@@ -256,43 +234,135 @@
     </gazebo>
     <!-- Camera sensor -->
-    <gazebo reference="camera_link">
-        <sensor name="${robot_name}" type="depth">
-            <update_rate>10.0</update_rate>
-            <camera name="${robot_name}_camera">
-                <horizontal_fov>1.047198</horizontal_fov>
-                <image>
-                    <width>640</width>
-                    <height>480</height>
-                    <format>R8G8B8</format>
-                </image>
-                <clip>
-                    <near>0.05</near>
-                    <far>3</far>
-                </clip>
-            </camera>
-            <plugin name="${robot_name}_camera_plugin" filename="libgazebo_ros_camera.so">
-                <baseline>0.2</baseline>
-                <alwaysOn>true</alwaysOn>
-                <updateRate>0.0</updateRate>
-                <!-- <imageTopicName>/${robot_name}/color/image_raw</imageTopicName>
-                <cameraInfoTopicName>/${robot_name}/color/camera_info</cameraInfoTopicName>
-                <depthImageTopicName>/${robot_name}/depth/image_raw</depthImageTopicName>
-                <depthImageInfoTopicName>/${robot_name}/depth/camera_info</depthImageInfoTopicName>
-                <pointCloudTopicName>/${robot_name}/depth/points</pointCloudTopicName> -->
-                <frameName>${robot_name}/camera_link</frameName>
-                <pointCloudCutoff>0.5</pointCloudCutoff>
-                <pointCloudCutoffMax>3.0</pointCloudCutoffMax>
-                <distortionK1>0.00000001</distortionK1>
-                <distortionK2>0.00000001</distortionK2>
-                <distortionK3>0.00000001</distortionK3>
-                <distortionT1>0.00000001</distortionT1>
-                <distortionT2>0.00000001</distortionT2>
-                <CxPrime>0</CxPrime>
-                <Cx>0</Cx>
-                <Cy>0</Cy>
-                <focalLength>0</focalLength>
-                <hackBaseline>0</hackBaseline>
-            </plugin>
-        </sensor>
-    </gazebo>
+   <gazebo reference="camera_link">
+    <sensor name="cameradepth" type="depth">
+        <camera name="camera">
+          <horizontal_fov>1.57</horizontal_fov>
+          <image>
+            <width>1280</width>
+            <height>720</height>
+          </image>
+          <clip>
+            <near>0.1</near>
+            <far>100</far>
+          </clip>
+          <noise>
+            <type>gaussian</type>
+            <mean>0.0</mean>
+            <stddev>0.100</stddev>
+          </noise>
+        </camera>
+        <always_on>1</always_on>
+        <update_rate>30</update_rate>
+        <visualize>0</visualize>
+      </sensor>
+      <sensor name="cameracolor" type="camera">
+        <camera name="camera">
+          <horizontal_fov>1.57</horizontal_fov>
+          <image>
+            <width>1280</width>
+            <height>720</height>
+            <format>RGB_INT8</format>
+          </image>
+          <clip>
+            <near>0.1</near>
+            <far>100</far>
+          </clip>
+          <noise>
+            <type>gaussian</type>
+            <mean>0.0</mean>
+            <stddev>0.007</stddev>
+          </noise>
+        </camera>
+        <always_on>1</always_on>
+        <update_rate>30</update_rate>
+        <visualize>1</visualize>
+      </sensor>
+      <sensor name="cameraired1" type="camera">
+        <camera name="camera">
+          <horizontal_fov>1.57</horizontal_fov>
+          <image>
+            <width>1280</width>
+            <height>720</height>
+            <format>L_INT8</format>
+          </image>
+          <clip>
+            <near>0.1</near>
+            <far>100</far>
+          </clip>
+          <noise>
+            <type>gaussian</type>
+            <mean>0.0</mean>
+            <stddev>0.05</stddev>
+          </noise>
+        </camera>
+        <always_on>1</always_on>
+        <update_rate>1</update_rate>
+        <visualize>0</visualize>
+      </sensor>
+      <sensor name="cameraired2" type="camera">
+        <camera name="camera">
+          <horizontal_fov>1.57</horizontal_fov>
+          <image>
+            <width>1280</width>
+            <height>720</height>
+            <format>L_INT8</format>
+          </image>
+          <clip>
+            <near>0.1</near>
+            <far>100</far>
+          </clip>
+          <noise>
+            <type>gaussian</type>
+            <mean>0.0</mean>
+            <stddev>0.05</stddev>
+          </noise>
+        </camera>
+        <always_on>1</always_on>
+        <update_rate>1</update_rate>
+        <visualize>0</visualize>
+      </sensor>
+   </gazebo>
+   <gazebo>
+    <plugin name="${robot_name}_camera" filename="librealsense_gazebo_plugin.so">
+        <prefix>camera</prefix>
+        <!--
+            actual FPS (and publishing rate, Hz) is 6 (at 1280x720) for realsense depth module.
+            Plugin caps depth FPS at 6. To increase FPS, decrease resolution in cameradepth sensor tag
+            Possible combinations for D435i:
+                1280x720x6
+                256x144x90
+                480x270x15
+                480x270x30
+                480x270x6
+                480x270x60
+                640x360x30
+                640x480x15
+                640x480x30
+                640x480x6
+                848x480x10
+                848x480x6
+                848x480x8
+        -->
+        <depthUpdateRate>30.0</depthUpdateRate>
+        <colorUpdateRate>30.0</colorUpdateRate>
+        <infraredUpdateRate>1.0</infraredUpdateRate>
+        <depthTopicName>${robot_name}/camera/depth/image_raw</depthTopicName>
+      	<depthCameraInfoTopicName>${robot_name}/camera/depth/camera_info</depthCameraInfoTopicName>
+      	<colorTopicName>${robot_name}/camera/color/image_raw</colorTopicName>
+      	<colorCameraInfoTopicName>${robot_name}/camera/color/camera_info</colorCameraInfoTopicName>
+      	<infrared1TopicName>${robot_name}/camera/infra1/image_raw</infrared1TopicName>
+      	<infrared1CameraInfoTopicName>${robot_name}/camera/infra1/camera_info</infrared1CameraInfoTopicName>
+      	<infrared2TopicName>${robot_name}/infra2/image_raw</infrared2TopicName>
+      	<infrared2CameraInfoTopicName>${robot_name}/camera/infra2/camera_info</infrared2CameraInfoTopicName>
+        <colorOpticalframeName>${robot_name}/camera_color_optical_frame</colorOpticalframeName>
+        <depthOpticalframeName>${robot_name}/camera_depth_optical_frame</depthOpticalframeName>
+        <infrared1OpticalframeName>${robot_name}/camera_left_ir_optical_frame</infrared1OpticalframeName>
+        <infrared2OpticalframeName>${robot_name}/camera_right_ir_optical_frame</infrared2OpticalframeName>
+        <rangeMinDepth>0.3</rangeMinDepth>
+        <rangeMaxDepth>3.0</rangeMaxDepth>
+        <pointCloud>true</pointCloud>
+        <pointCloudTopicName>${robot_name}/camera/depth/points</pointCloudTopicName>
+        <pointCloudCutoff>0.3</pointCloudCutoff>
+    </plugin>
+   </gazebo>
 </robot>

Commit message: feat: added ros2 control for real robot case

File: xacro/vikings_bot.xacro (robot description, xacro)
@@ -3,8 +3,8 @@
     <!-- Argumnets -->
     <xacro:arg name="vikings_bot_name" default="vikings_bot"/>
-    <xacro:arg name="use_gazebo" default="yes"/>
+    <xacro:arg name="use_sim" default="true"/>
     <!-- Robot properties -->
     <xacro:property name="robot_name" value="$(arg vikings_bot_name)"/>
-    <xacro:property name="use_gazebo" value="$(arg use_gazebo)"/>
+    <xacro:property name="use_sim" value="$(arg use_sim)"/>
     <!-- Include robot properties -->
     <xacro:include filename="$(find vikings_bot_description)/xacro/properties.xacro"/>
@@ -14,6 +14,4 @@
     <xacro:include filename="$(find vikings_bot_description)/xacro/wheels.xacro"/>
     <xacro:include filename="$(find vikings_bot_description)/xacro/castor_wheels.xacro"/>
-    <!-- Inlude gazebo stuff -->
-    <!-- <xacro:include filename="$(find vikings_bot_description)/xacro/gazebo_plugins.xacro"/> -->
     <!-- Include Gazebo related files -->
     <!-- ROBOT -->
@@ -176,47 +174,15 @@
         <origin xyz="${camera_xoff} ${camera_yoff} ${camera_zoff}" rpy="0 0 0"/>
     </joint>
-    <!-- PLUGINS -->
-    <gazebo>
-        <plugin name="${robot_name}_joint_state" filename="libgazebo_ros_joint_state_publisher.so">
-            <ros>
-                <namespace>/${robot_name}</namespace>
-                <!-- <remapping>~/out:=joint_states</remapping> -->
-            </ros>
-            <update_rate>30</update_rate>
-            <joint_name>left_drive_wheel_joint</joint_name>
-            <joint_name>right_drive_wheel_joint</joint_name>
-            <joint_name>left_castor_wheel_yaw_joint</joint_name>
-            <joint_name>right_castor_wheel_yaw_joint</joint_name>
-            <joint_name>left_castor_wheel_pitch_joint</joint_name>
-            <joint_name>right_castor_wheel_pitch_joint</joint_name>
-        </plugin>
-    </gazebo>
-    <!-- Differential drive -->
-    <gazebo>
-        <plugin filename="libgazebo_ros_diff_drive.so" name="${robot_name}_differential_drive_controller">
-        <ros>
-            <namespace>/${robot_name}</namespace>
-            <!--
-    <argument> -ros-args -remap /cmd_vel:=/${robot_name}/cmd_vel /odom:=/${robot_name}/odom</argument>
--->
-        </ros>
-        <!-- wheels -->
-        <!-- wheels RMF COMPAT -->
-        <left_joint>left_drive_wheel_joint</left_joint>
-        <right_joint>right_drive_wheel_joint</right_joint>
-        <!-- kinematics -->
-        <wheel_separation>${wheel_yoff * 2}</wheel_separation>
-        <wheel_diameter>${wheel_radius * 2}</wheel_diameter>
-        <!-- limits -->
-        <max_wheel_torque>10000</max_wheel_torque>
-        <max_wheel_acceleration>1000</max_wheel_acceleration>
-        <!-- output -->
-        <publish_odom>true</publish_odom>
-        <publish_odom_tf>true</publish_odom_tf>
-        <!-- <publish_wheel_tf>false</publish_wheel_tf> -->
-        <odometry_frame>${robot_name}/odom</odometry_frame>
-        <robot_base_frame>${robot_name}/dummy_link</robot_base_frame>
-        </plugin>
-    </gazebo>
+    <!-- If use "use_sim "-->
+    <xacro:if value="${use_sim}">
+        <!-- Inlude gazebo stuff -->
+        <xacro:include filename="$(find vikings_bot_description)/xacro/gazebo_control.xacro"/>
+    </xacro:if>
+    <!-- If not use "use_sim "-->
+    <xacro:unless value="${use_sim}">
+        <!-- Inlude gazebo stuff -->
+        <xacro:include filename="$(find vikings_bot_description)/xacro/ros2_control.xacro"/>
+        <xacro:diffdrive_ros2_control name="${robot_name}" use_mock_hardware="false"/>
+    </xacro:unless>
     <!-- Lidar  sensor -->
     <gazebo reference="lidar_link">

Commit message: added realsense gazebo plugin & realsense_2_description

File: xacro/vikings_bot.xacro (robot description, xacro)
@@ -14,4 +14,5 @@
     <xacro:include filename="$(find vikings_bot_description)/xacro/wheels.xacro"/>
     <xacro:include filename="$(find vikings_bot_description)/xacro/castor_wheels.xacro"/>
+    <xacro:include filename="$(find realsense2_description)/urdf/_d415.urdf.xacro"/>
     <!-- Include Gazebo related files -->
     <!-- ROBOT -->
@@ -121,25 +122,9 @@
     </joint>
     <!-- Camera -->
-    <link name="camera_link">
-        <visual>
-            <origin xyz="0 0 0" rpy="0 0 ${1.57*2}"/>
-            <geometry>
-                <mesh filename="package://vikings_bot_description/meshes/sensors/realsense.dae"
-                      scale="1 1 1"/>
-            </geometry>
-        </visual>
-        <inertial>
-            <mass value="0.2"/>
-            <origin xyz=" 0 0 0" rpy="0 0 0" />
-            <inertia ixx="1e-7" ixy="0" ixz="0"
-                     iyx="0" iyy="1e-7" iyz="0"
-                     izx="0" izy="0" izz="1e-7" />
-        </inertial>
-        <collision>
-            <geometry>
-                <box size="0.08 0.1 0.03"/>
-            </geometry>
-        </collision>
-    </link>
+    <!-- realsense2_description package manages camera's description (geometry etc.) -->
+    <!--TODO: add use sim time parameter to use_nominal_extrinsics (should only be true in sim)-->
+    <xacro:sensor_d415 parent="chassis_link" use_nominal_extrinsics="${use_sim}">
+        <origin xyz="${camera_xoff} ${camera_yoff} ${camera_zoff}" rpy="0 0 0"/>
+    </xacro:sensor_d415>
     <gazebo reference="camera_link">
         <material>Gazebo/Grey</material>
@@ -151,9 +136,4 @@
         <kd>100000000000000000</kd>
     </gazebo>
-    <joint name="camera_link_joint" type="fixed">
-        <parent link="chassis_link"/>
-        <child link="camera_link"/>
-        <origin xyz="${camera_xoff} ${camera_yoff} ${camera_zoff}" rpy="0 0 0"/>
-    </joint>
     <!-- If use "use_sim "-->
     <xacro:if value="${use_sim}">
@@ -203,44 +183,127 @@
         </sensor>
     </gazebo>
-    <!-- Camera sensor -->
-    <gazebo reference="camera_link">
-        <sensor name="${robot_name}" type="depth">
-            <update_rate>10.0</update_rate>
-            <camera name="${robot_name}_camera">
-                <horizontal_fov>1.047198</horizontal_fov>
-                <image>
-                    <width>640</width>
-                    <height>480</height>
-                    <format>R8G8B8</format>
-                </image>
-                <clip>
-                    <near>0.05</near>
-                    <far>3</far>
-                </clip>
-            </camera>
-            <plugin name="${robot_name}_camera_plugin" filename="libgazebo_ros_camera.so">
-                <baseline>0.2</baseline>
-                <alwaysOn>true</alwaysOn>
-                <updateRate>0.0</updateRate>
-                <!-- <imageTopicName>/${robot_name}/color/image_raw</imageTopicName>
-                <cameraInfoTopicName>/${robot_name}/color/camera_info</cameraInfoTopicName>
-                <depthImageTopicName>/${robot_name}/depth/image_raw</depthImageTopicName>
-                <depthImageInfoTopicName>/${robot_name}/depth/camera_info</depthImageInfoTopicName>
-                <pointCloudTopicName>/${robot_name}/depth/points</pointCloudTopicName> -->
-                <frameName>${robot_name}/camera_link</frameName>
-                <pointCloudCutoff>0.5</pointCloudCutoff>
-                <pointCloudCutoffMax>3.0</pointCloudCutoffMax>
-                <distortionK1>0.00000001</distortionK1>
-                <distortionK2>0.00000001</distortionK2>
-                <distortionK3>0.00000001</distortionK3>
-                <distortionT1>0.00000001</distortionT1>
-                <distortionT2>0.00000001</distortionT2>
-                <CxPrime>0</CxPrime>
-                <Cx>0</Cx>
-                <Cy>0</Cy>
-                <focalLength>0</focalLength>
-                <hackBaseline>0</hackBaseline>
-            </plugin>
-        </sensor>
-    </gazebo>
+   <!-- Camera sensor -->
+   <!--
+    uses pal robotics realsense_gazebo_plugin
+    https://github.com/pal-robotics/realsense_gazebo_plugin/tree/foxy-devel
+   -->
+   <gazebo reference="camera_link">
+    <sensor name="cameradepth" type="depth">
+        <camera name="camera">
+          <horizontal_fov>1.57</horizontal_fov>
+          <image>
+            <width>${camera_depth_width}</width>
+            <height>${camera_depth_height}</height>
+          </image>
+          <clip>
+            <near>0.1</near>
+            <far>100</far>
+          </clip>
+          <noise>
+            <type>gaussian</type>
+            <mean>0.0</mean>
+            <stddev>0.100</stddev>
+          </noise>
+        </camera>
+        <always_on>1</always_on>
+        <update_rate>30</update_rate>
+        <visualize>0</visualize>
+      </sensor>
+      <sensor name="cameracolor" type="camera">
+        <camera name="camera">
+          <horizontal_fov>1.57</horizontal_fov>
+          <image>
+            <width>${camera_color_width}</width>
+            <height>${camera_color_height}</height>
+            <format>RGB_INT8</format>
+          </image>
+          <clip>
+            <near>0.1</near>
+            <far>100</far>
+          </clip>
+          <noise>
+            <type>gaussian</type>
+            <mean>0.0</mean>
+            <stddev>0.007</stddev>
+          </noise>
+        </camera>
+        <always_on>1</always_on>
+        <update_rate>30</update_rate>
+        <visualize>1</visualize>
+      </sensor>
+      <sensor name="cameraired1" type="camera">
+        <camera name="camera">
+          <horizontal_fov>1.57</horizontal_fov>
+          <image>
+            <width>${camera_depth_width}</width>
+            <height>${camera_depth_height}</height>
+            <format>L_INT8</format>
+          </image>
+          <clip>
+            <near>0.1</near>
+            <far>100</far>
+          </clip>
+          <noise>
+            <type>gaussian</type>
+            <mean>0.0</mean>
+            <stddev>0.05</stddev>
+          </noise>
+        </camera>
+        <always_on>1</always_on>
+        <update_rate>1</update_rate>
+        <visualize>0</visualize>
+      </sensor>
+      <sensor name="cameraired2" type="camera">
+        <camera name="camera">
+          <horizontal_fov>1.57</horizontal_fov>
+          <image>
+            <width>${camera_depth_width}</width>
+            <height>${camera_depth_height}</height>
+            <format>L_INT8</format>
+          </image>
+          <clip>
+            <near>0.1</near>
+            <far>100</far>
+          </clip>
+          <noise>
+            <type>gaussian</type>
+            <mean>0.0</mean>
+            <stddev>0.05</stddev>
+          </noise>
+        </camera>
+        <always_on>1</always_on>
+        <update_rate>1</update_rate>
+        <visualize>0</visualize>
+      </sensor>
+   </gazebo>
+   <gazebo>
+    <plugin name="${robot_name}_camera" filename="librealsense_gazebo_plugin.so">
+        <prefix>camera</prefix>
+        <!--
+            actual FPS (and publishing rate, Hz) is 6 (at 1280x720) for realsense depth module.
+            Plugin caps depth FPS at 6. To increase FPS, change resolution in properties.xacro
+        -->
+        <depthUpdateRate>30.0</depthUpdateRate>
+        <colorUpdateRate>30.0</colorUpdateRate>
+        <infraredUpdateRate>1.0</infraredUpdateRate>
+        <depthTopicName>${robot_name}/camera/depth/image_rect_raw</depthTopicName>
+      	<depthCameraInfoTopicName>${robot_name}/camera/depth/camera_info</depthCameraInfoTopicName>
+      	<colorTopicName>${robot_name}/camera/color/image_raw</colorTopicName>
+      	<colorCameraInfoTopicName>${robot_name}/camera/color/camera_info</colorCameraInfoTopicName>
+        <!--real realsense camera does not publish infared image topics, but removing these params breaks the plugin-->
+      	<infrared1TopicName>${robot_name}/camera/infra1/image_raw</infrared1TopicName>
+      	<infrared1CameraInfoTopicName>${robot_name}/camera/infra1/camera_info</infrared1CameraInfoTopicName>
+      	<infrared2TopicName>${robot_name}/infra2/image_raw</infrared2TopicName>
+      	<infrared2CameraInfoTopicName>${robot_name}/camera/infra2/camera_info</infrared2CameraInfoTopicName>
+        <colorOpticalframeName>${robot_name}/camera_color_optical_frame</colorOpticalframeName>
+        <depthOpticalframeName>${robot_name}/camera_depth_optical_frame</depthOpticalframeName>
+        <infrared1OpticalframeName>${robot_name}/camera_left_ir_optical_frame</infrared1OpticalframeName>
+        <infrared2OpticalframeName>${robot_name}/camera_right_ir_optical_frame</infrared2OpticalframeName>
+        <rangeMinDepth>0.3</rangeMinDepth>
+        <rangeMaxDepth>3.0</rangeMaxDepth>
+        <pointCloud>true</pointCloud>
+        <pointCloudTopicName>${robot_name}/camera/depth/color/points</pointCloudTopicName>
+        <pointCloudCutoff>0.3</pointCloudCutoff>
+    </plugin>
+   </gazebo>
 </robot>
