Commit message: correct camera offset

File: xacro/properties.xacro (robot description, xacro)
@@ -26,5 +26,5 @@
     <xacro:property name="lidar_zoff" value="-0.06"/>
     <!-- Camera -->
-    <xacro:property name="camera_xoff" value="0.5"/>
+    <xacro:property name="camera_xoff" value="0.51"/>
     <xacro:property name="camera_yoff" value="0.0"/>
     <xacro:property name="camera_zoff" value="0.06"/>

Commit message: added setting to change camera resolution

File: xacro/properties.xacro (robot description, xacro)
@@ -29,3 +29,26 @@
     <xacro:property name="camera_yoff" value="0.0"/>
     <xacro:property name="camera_zoff" value="0.06"/>
+    <xacro:property name="camera_depth_width" value="1280"/>
+    <xacro:property name="camera_depth_height" value="720"/>
+    <xacro:property name="camera_color_width" value="1280"/>
+    <xacro:property name="camera_color_height" value="720"/>
+    <!--
+        Possible depth resolutions for D435i (maximum FPS for resolution is default):
+                1280x720 -> 6 FPS
+                256x144 -> 90 FPS
+                480x270 -> 15 FPS
+                480x270 -> 30 FPS
+                480x270 -> 6 FPS
+                480x270 -> 60 FPS
+                640x360 -> 30 FPS
+                640x480 -> 15 FPS
+                640x480 -> 30 FPS
+                640x480 -> 6 FPS
+                848x480 -> 10 FPS
+                848x480 -> 6 FPS
+                848x480 -> 8 FPS
+        BUG: Changing camera_depth* yields Gazebo error:
+            terminate called after throwing an instance of 'std::runtime_error'
+            [gzserver-1]   what():  unsupported colour encoding: 8UC1
+    -->
 </robot>

File: xacro/vikings_bot.xacro (robot description, xacro)
@@ -239,6 +239,6 @@
           <horizontal_fov>1.57</horizontal_fov>
           <image>
-            <width>1280</width>
-            <height>720</height>
+            <width>${camera_depth_width}</width>
+            <height>${camera_depth_height}</height>
           </image>
           <clip>
@@ -260,6 +260,6 @@
           <horizontal_fov>1.57</horizontal_fov>
           <image>
-            <width>1280</width>
-            <height>720</height>
+            <width>${camera_color_width}</width>
+            <height>${camera_color_height}</height>
             <format>RGB_INT8</format>
           </image>
@@ -328,19 +328,5 @@
         <!--
             actual FPS (and publishing rate, Hz) is 6 (at 1280x720) for realsense depth module.
-            Plugin caps depth FPS at 6. To increase FPS, decrease resolution in cameradepth sensor tag
-            Possible combinations for D435i:
-                1280x720x6
-                256x144x90
-                480x270x15
-                480x270x30
-                480x270x6
-                480x270x60
-                640x360x30
-                640x480x15
-                640x480x30
-                640x480x6
-                848x480x10
-                848x480x6
-                848x480x8
+            Plugin caps depth FPS at 6. To increase FPS, change resolution in properties.xacro
         -->
         <depthUpdateRate>30.0</depthUpdateRate>

Commit message: changed camera resolution

File: xacro/properties.xacro (robot description, xacro)
@@ -30,8 +30,8 @@
     <xacro:property name="camera_yoff" value="0.0"/>
     <xacro:property name="camera_zoff" value="0.06"/>
-    <xacro:property name="camera_depth_width" value="1280"/>
-    <xacro:property name="camera_depth_height" value="720"/>
-    <xacro:property name="camera_color_width" value="1280"/>
-    <xacro:property name="camera_color_height" value="720"/>
+    <xacro:property name="camera_depth_width" value="640"/>
+    <xacro:property name="camera_depth_height" value="480"/>
+    <xacro:property name="camera_color_width" value="640"/>
+    <xacro:property name="camera_color_height" value="480"/>
     <!--
         Possible depth resolutions for D435i (maximum FPS for resolution is default):
@@ -49,7 +49,16 @@
                 848x480 -> 6 FPS
                 848x480 -> 8 FPS
-        BUG: Changing camera_depth* yields Gazebo error:
-            terminate called after throwing an instance of 'std::runtime_error'
-            [gzserver-1]   what():  unsupported colour encoding: 8UC1
+        Possible rgb resolutions for D435i:
+                1280x720 -> 10
+                1280x720 -> 15
+                1280x720 -> 6
+                1920x1080 -> 8
+                424x240 -> 15
+                424x240 -> 30
+                424x240 -> 6
+                424x240 -> 60
+                640x480 -> 15
+                640x480 -> 30
+                640x480 -> 6
     -->
 </robot>

File: xacro/vikings_bot.xacro (robot description, xacro)
@@ -282,6 +282,6 @@
           <horizontal_fov>1.57</horizontal_fov>
           <image>
-            <width>1280</width>
-            <height>720</height>
+            <width>${camera_depth_width}</width>
+            <height>${camera_depth_height}</height>
             <format>L_INT8</format>
           </image>
@@ -304,6 +304,6 @@
           <horizontal_fov>1.57</horizontal_fov>
           <image>
-            <width>1280</width>
-            <height>720</height>
+            <width>${camera_depth_width}</width>
+            <height>${camera_depth_height}</height>
             <format>L_INT8</format>
           </image>

Commit message: added camera res params

File: xacro/properties.xacro (robot description, xacro)
@@ -27,6 +27,10 @@
     <!-- <xacro:property name="lidar_zoff" value="-0.06"/> -->
     <!-- Camera -->
-    <xacro:property name="camera_xoff" value="0.5"/>
+    <xacro:property name="camera_xoff" value="0.51"/>
     <xacro:property name="camera_yoff" value="0.0"/>
     <xacro:property name="camera_zoff" value="0.06"/>
+    <xacro:property name="camera_depth_width" value="640"/>
+    <xacro:property name="camera_depth_height" value="480"/>
+    <xacro:property name="camera_color_width" value="640"/>
+    <xacro:property name="camera_color_height" value="480"/>
 </robot>

Commit message: remeasured lidar and camera offsets

File: xacro/properties.xacro (robot description, xacro)
@@ -22,12 +22,12 @@
     <xacro:property name="castor_wheel_width" value="0.05"/>
     <!-- Lidar -->
-    <xacro:property name="lidar_xoff" value="0.53"/>
+    <xacro:property name="lidar_xoff" value="0.495"/>
     <xacro:property name="lidar_yoff" value="0.0"/>
-    <xacro:property name="lidar_zoff" value="-0.02"/>
+    <xacro:property name="lidar_zoff" value="-0.0273"/>
     <!-- <xacro:property name="lidar_zoff" value="-0.06"/> -->
     <!-- Camera -->
-    <xacro:property name="camera_xoff" value="0.51"/>
+    <xacro:property name="camera_xoff" value="0.4972"/>
     <xacro:property name="camera_yoff" value="0.0"/>
-    <xacro:property name="camera_zoff" value="0.06"/>
+    <xacro:property name="camera_zoff" value="0.0298"/>
     <xacro:property name="camera_depth_width" value="640"/>
     <xacro:property name="camera_depth_height" value="480"/>

Commit message: updated lidar position

File: xacro/properties.xacro (robot description, xacro)
@@ -22,5 +22,5 @@
     <xacro:property name="castor_wheel_width" value="0.05"/>
     <!-- Lidar -->
-    <xacro:property name="lidar_xoff" value="0.495"/>
+    <xacro:property name="lidar_xoff" value="0.51"/>
     <xacro:property name="lidar_yoff" value="0.0"/>
     <xacro:property name="lidar_zoff" value="-0.0273"/>
